File: OpenDropV2.kicad_pcb (KiCad board)
At the start: 2 copper layers, 100 x 100 mm, 200 parts, among them J1 DC_JACK, P1 CONN_01X01, P2 CONN_01X01, P3 CONN_01X01, P4 CONN_01X01, P5 CONN_01X01, Q1 BSS138, Q2 BSS138, Q3 BSS138, SW1 SW_PUSH, SW2 SW_PUSH, SW3 SW_PUSH, SW4 SW_PUSH, SW5 SPST, T1 IRF 840S, U1 MAX1771ESA, U2 HV507, U3 ARDUINO_MICRO, U4 HV507, U5 ESP8266_SMD

Commit message: started with corrections for V2.1
work in progress
Parts:
- C6: footprint Resistors_SMD:R_2512 -> GaudiLabsFootPrints:C100n_250V
- D1: footprint Diodes_SMD:DO-214AB -> GaudiLabsFootPrints:DO-214AA
- D2, D3, D4: value D_Small -> 1N4148
- POT1: value POT -> 5k Ohm
- R5: value 390 -> 10
- U1: footprint SMD_Packages:SOIC-8-N -> GaudiLabsFootPrints:SO08
- moved C6 22.0 mm to (87.7, 49.1), turned to 0 degrees
- moved LED5 17.2 mm to (102.2, 73.4)
- moved D4 7.95 mm to (146.1, 52.9), turned to 270 degrees
- moved D2 7.45 mm to (148.1, 52.9), turned to 270 degrees
- moved D1 6.33 mm to (95.9, 51.0), turned to 90 degrees
- moved C2 4.44 mm to (74.6, 69.0)
- moved R8 3.46 mm to (124.5, 58.2)
- moved R14 3.06 mm to (129.3, 53.4)
- moved R11 3.06 mm to (127.3, 53.4)
- moved R13 3.05 mm to (134.4, 53.4)
- moved C9 2.31 mm to (123.2, 53.4)
- moved C4 2.00 mm to (74.9, 51.2)
- moved L1 2.00 mm to (90.1, 76.1)
- moved T1 2.00 mm to (84.8, 62.1)
- moved U1 2.00 mm to (79.2, 62.9)
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Connections:
- POT1 pad 1: V_READ_HV -> Net-(POT1-Pad1)
- POT1 pad 2: Net-(POT1-Pad2) -> Net-(POT1-Pad1)
- POT1 pad 3: Net-(POT1-Pad2) -> V_READ_HV
- R1 pad 1: Net-(POT1-Pad2) -> Net-(POT1-Pad1)
Routing:
- net (no net): track 0.02 -> 269.8 mm, vias 0 -> 3
- net SW2: track 85.3 -> 14.8 mm
- net SW1: track 157.1 -> 91.5 mm
- net SW4: track 101.4 -> 36.0 mm
- net SW3: track 137.8 -> 72.6 mm
- net V_HV: track 149.7 -> 165.5 mm
- net Net-(LED2-Pad2): track 172.4 -> 157.9 mm, vias 9 -> 7
- net Net-(POT1-Pad1): track 0.00 -> 13.5 mm, vias 0 -> 1
- net GND: track 381.1 -> 368.7 mm, vias 12 -> 9
- net Net-(D4-Pad2): track 20.6 -> 32.6 mm
- net Net-(POT1-Pad2): track 10.7 -> 0.00 mm
- net Net-(D2-Pad2): track 29.1 -> 39.2 mm
- net Net-(P1-Pad1): track 9.92 -> 0.00 mm
- net +5V: track 193.5 -> 202.5 mm
- net 3.3V: track 85.8 -> 94.1 mm
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Other:
- outline, holes or cut-outs redrawn

Commit message: More modifications and corrections for Version 2.1
work in progress
Parts:
- removed LED6, LED7: LED, GaudiLabsFootPrints:LED_SIDE
- removed SW3, SW4: SW_PUSH, Buttons_Switches_SMD:SW_SPST_PTS645
- added JS1: JoystickSMD, GaudiLabsFootPrints:JoystickSMD_SKQUSeries, F.Cu at (100.0, 136.4)
- added P6: CONN_01X30, GaudiLabsFootPrints:OLED_SolderPads, F.Cu at (131.8, 61.7)
- added R18: 10k, Resistors_SMD:R_0805, B.Cu at (102.4, 135.9)
- added R19: 10k, Resistors_SMD:R_0805, B.Cu at (100.0, 135.9)
- added R20: 10k, Resistors_SMD:R_0805, B.Cu at (97.3, 137.4)
- added R21: 10k, Resistors_SMD:R_0805, B.Cu at (97.3, 134.0)
- added REF**: Fiducial_1mm_Dia_2.54mm_Outer_CopperBottom, Fiducials:Fiducial_1mm_Dia_2.54mm_Outer_CopperBottom, F.Cu at (53.0, 133.0)
- added REF**: Fiducial_1mm_Dia_2.54mm_Outer_CopperTop, Fiducials:Fiducial_1mm_Dia_2.54mm_Outer_CopperTop, F.Cu at (147.0, 133.0)
- added REF**: Fiducial_1mm_Dia_2.54mm_Outer_CopperBottom, Fiducials:Fiducial_1mm_Dia_2.54mm_Outer_CopperBottom, F.Cu at (147.0, 45.0)
- added REF**: Fiducial_1mm_Dia_2.54mm_Outer_CopperTop, Fiducials:Fiducial_1mm_Dia_2.54mm_Outer_CopperTop, F.Cu at (147.0, 45.0)
- added REF**: Fiducial_1mm_Dia_2.54mm_Outer_CopperTop, Fiducials:Fiducial_1mm_Dia_2.54mm_Outer_CopperTop, F.Cu at (53.0, 133.0)
- added REF**: Fiducial_1mm_Dia_2.54mm_Outer_CopperBottom, Fiducials:Fiducial_1mm_Dia_2.54mm_Outer_CopperBottom, F.Cu at (147.0, 133.0)
- FLUXL1, FLUXL10, FLUXL100, FLUXL101, FLUXL102, FLUXL103, FLUXL104, FLUXL105, FLUXL106, FLUXL107, FLUXL108, FLUXL109, FLUXL11, FLUXL110, FLUXL111, FLUXL112, FLUXL113, FLUXL114, FLUXL115, FLUXL116, FLUXL117, FLUXL118, FLUXL119, FLUXL12, FLUXL120, FLUXL121, FLUXL122, FLUXL123, FLUXL124, FLUXL125, FLUXL126, FLUXL127, FLUXL128, FLUXL13, FLUXL14, FLUXL15, FLUXL16, FLUXL17, FLUXL18, FLUXL19, FLUXL2, FLUXL20, FLUXL21, FLUXL22, FLUXL23, FLUXL24, FLUXL25, FLUXL26, FLUXL27, FLUXL28, FLUXL29, FLUXL3, FLUXL30, FLUXL31, FLUXL32, FLUXL33, FLUXL34, FLUXL35, FLUXL36, FLUXL37, FLUXL38, FLUXL39, FLUXL4, FLUXL40, FLUXL41, FLUXL42, FLUXL43, FLUXL44, FLUXL45, FLUXL46, FLUXL47, FLUXL48, FLUXL49, FLUXL5, FLUXL50, FLUXL51, FLUXL52, FLUXL53, FLUXL54, FLUXL55, FLUXL56, FLUXL57, FLUXL58, FLUXL59, FLUXL6, FLUXL60, FLUXL61, FLUXL62, FLUXL63, FLUXL64, FLUXL65, FLUXL66, FLUXL67, FLUXL68, FLUXL69, FLUXL7, FLUXL70, FLUXL71, FLUXL72, FLUXL73, FLUXL74, FLUXL75, FLUXL76, FLUXL77, FLUXL78, FLUXL79, FLUXL8, FLUXL80, FLUXL81, FLUXL82, FLUXL83, FLUXL84, FLUXL85, FLUXL86, FLUXL87, FLUXL88, FLUXL89, FLUXL9, FLUXL90, FLUXL91, FLUXL92, FLUXL93, FLUXL94, FLUXL95, FLUXL96, FLUXL97, FLUXL98, FLUXL99: footprint GaudiLabsFootPrints:FLUXL_PAD_2_75 -> GaudiLabsFootPrints:FLUXPAD_2_75_4MIL_4_5
- SW1, SW2: footprint Buttons_Switches_SMD:SW_SPST_PTS645 -> GaudiLabsFootPrints:PUSH_BUTTON_SMD
- U2, U4: footprint Housings_QFP:PQFP-80_14x20mm_Pitch0.8mm -> GaudiLabsFootPrints:PQFP-80_14x20mm_Pitch0.8mm
- moved LED4 69.9 mm to (89.0, 67.2), turned to 180 degrees
- moved LED2 25.0 mm to (111.0, 131.8)
- moved LED3 11.0 mm to (89.0, 131.8)
- moved LED5 10.8 mm to (111.0, 67.2)
- turned SW1 to 180 degrees
- turned SW2 to 180 degrees
Connections:
- net DI1 renamed DI
- U2 pad 26: DI2 -> Net-(U2-Pad26)
- U2 pad 29: +5V -> BL
- U2 pad 30: POL -> +5V
- U3 pad 25: SW4 -> JOY
- U3 pad 7: DI2 -> (no net)
- U3 pad 8: POL -> BL
- U4 pad 29: +5V -> BL
- U4 pad 30: POL -> +5V
- U4 pad 39: (no net) -> Net-(U2-Pad26)
Routing:
- net (no net): track 269.8 -> 22.5 mm
- net POL: track 165.5 -> 0.00 mm, vias 2 -> 0
- net Net-(U2-Pad26): track 0.00 -> 118.3 mm
- net DI2: track 118.3 -> 0.00 mm
- net JOY: track 0.00 -> 105.7 mm, vias 0 -> 1
- net GND: track 368.7 -> 276.6 mm
- net +5V: track 202.5 -> 284.2 mm, vias 9 -> 6
- net BL: track 0.00 -> 66.8 mm, vias 0 -> 2
- net SW2: track 14.8 -> 80.4 mm
- net SW1: track 91.5 -> 155.4 mm
- net SW3: track 72.6 -> 131.0 mm
- net SW4: track 36.0 -> 0.00 mm, vias 1 -> 0
- net Net-(P6-Pad19): track 14.9 -> 43.7 mm, vias 2 -> 3
- net 3.3V: track 94.1 -> 103.6 mm
- net Net-(D4-Pad2): track 32.6 -> 41.5 mm, vias 2 -> 4
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Other:
- net class Big: clearance 0.2 -> 0.1524
- net class Default: clearance 0.2 -> 0.1524
- net class Power: clearance 0.2 -> 0.1524
- rule trace_clearance: 0.2 -> 0.1524

Commit message: Production Version of V2.1
Hopefully...
Parts:
- removed P4: CONN_01X01, Measurement_Points:Measurement_Point_Square-SMD-Pad_Small
- removed the REF** at (56.0, 74.0)
- removed the REF** at (56.0, 125.0)
- removed the REF** at (144.0, 125.0)
- removed the REF** at (144.0, 74.0)
- added C14: 100nF, Capacitors_SMD:C_0805, B.Cu at (143.6, 101.9)
- added C15: 1uF, Capacitors_SMD:C_0805, B.Cu at (118.4, 71.9)
- added C16: 1uF, Capacitors_SMD:C_0805, B.Cu at (115.1, 69.4)
- added C17: 1uF, Capacitors_SMD:C_0805, B.Cu at (110.5, 70.9)
- added D5: 1N4148, Diodes_SMD:SOD-323, B.Cu at (138.5, 101.9)
- added P10: CONN_01X01, Measurement_Points:Measurement_Point_Square-SMD-Pad_Small, B.Cu at (68.1, 105.9)
- added P11: CONN_01X01, Measurement_Points:Measurement_Point_Square-SMD-Pad_Small, B.Cu at (68.1, 98.3)
- added P12: CONN_01X01, Measurement_Points:Measurement_Point_Square-SMD-Pad_Small, B.Cu at (68.1, 100.9)
- added P13: ScrewPad1, GaudiLabsFootPrints:MountingHolePad_3x9mm, F.Cu at (144.0, 74.0)
- added P14: ScrewPad2, GaudiLabsFootPrints:MountingHolePad_3x9mm, F.Cu at (144.0, 125.0)
- added P15: ScrewPad3, GaudiLabsFootPrints:MountingHolePad_3x9mm, F.Cu at (56.0, 125.0)
- added P16: ScrewPad4, GaudiLabsFootPrints:MountingHolePad_3x9mm, F.Cu at (56.0, 74.0)
- added P7: CONN_01X01, Measurement_Points:Measurement_Point_Square-SMD-Pad_Small, B.Cu at (68.1, 108.5)
- added P8: CONN_01X01, Measurement_Points:Measurement_Point_Square-SMD-Pad_Small, B.Cu at (68.1, 95.8)
- added P9: CONN_01X01, Measurement_Points:Measurement_Point_Square-SMD-Pad_Small, B.Cu at (68.1, 93.2)
- added Q5: BSS138, TO_SOT_Packages_SMD:SOT-23, B.Cu at (141.5, 89.2)
- added Q6: BSS138, TO_SOT_Packages_SMD:SOT-23, B.Cu at (144.8, 89.2)
- added Q7: BSS138, TO_SOT_Packages_SMD:SOT-23, B.Cu at (137.7, 89.2)
- added R22: 10k, Resistors_SMD:R_0805, B.Cu at (118.9, 78.3)
- added R23: 10k, Resistors_SMD:R_0805, B.Cu at (141.5, 84.9)
- added R24: 10k, Resistors_SMD:R_0805, B.Cu at (135.7, 101.4)
- added R25: 10k, Resistors_SMD:R_0805, B.Cu at (144.8, 84.9)
- added R26: 10k, Resistors_SMD:R_0805, B.Cu at (147.6, 100.9)
- added R27: 10k, Resistors_SMD:R_0805, B.Cu at (136.7, 84.9)
- added R28: 10k, Resistors_SMD:R_0805, B.Cu at (138.7, 84.9)
- added R29: 10k, Resistors_SMD:R_0805, B.Cu at (146.9, 84.9)
- added R30: 10k, Resistors_SMD:R_0805, B.Cu at (118.4, 75.2)
- added R31: 10k, Resistors_SMD:R_0805, B.Cu at (110.5, 74.7)
- added U6: MCP6002, GaudiLabsFootPrints:SO08, B.Cu at (114.6, 75.0)
- P1: moved to F.Cu
- moved P3 74.0 mm to (68.1, 103.4)
- moved P1 9.23 mm to (144.6, 65.8)
- moved U5 9.03 mm to (140.8, 95.5)
- moved P2 1.90 mm to (135.9, 71.7)
- moved P5 0.51 mm to (147.4, 65.8)
Connections:
- P1 pad 1: Net-(P1-Pad1) -> V_GND
- P3 pad 1: Net-(P3-Pad1) -> +5V
- POT1 pad 3: V_READ_HV -> Net-(POT1-Pad3)
- R2 pad 2: V_READ_HV -> Net-(POT1-Pad3)
- U1 pad 3: V_READ_HV -> Net-(POT1-Pad3)
- U2 pad 39: (no net) -> DIO_B
- U3 pad 14: DISP_SDA -> BL
- U3 pad 15: DISP_SCL -> ESP_GPIO0
- U3 pad 21: V_READ_HV -> (no net)
- U3 pad 22: Net-(P1-Pad1) -> Net-(P2-Pad1)
- U3 pad 23: Net-(P2-Pad1) -> FEEDBACK
- U3 pad 24: Net-(P3-Pad1) -> ESP_RESET
- U3 pad 3: (no net) -> ESP_RX
- U3 pad 4: (no net) -> ESP_TX
- U3 pad 7: (no net) -> DISP_SDA
- U3 pad 8: BL -> DISP_SCL
- U5 pad 1: (no net) -> GND
- U5 pad 2: 3.3V -> Net-(Q6-Pad2)
- U5 pad 4: (no net) -> 3.3V
- U5 pad 5: (no net) -> Net-(Q5-Pad2)
- U5 pad 6: (no net) -> Net-(Q7-Pad2)
- U5 pad 7: GND -> Net-(D5-Pad2)
- U5 pad 8: (no net) -> 3.3V
Routing:
- net BL: track 66.8 -> 181.2 mm, vias 2 -> 4
- net +5V: track 284.2 -> 380.0 mm, vias 6 -> 8
- net ESP_TX: track 0.00 -> 81.3 mm, vias 0 -> 2
- net ESP_RX: track 0.00 -> 73.3 mm, vias 0 -> 2
- net 3.3V: track 103.6 -> 174.8 mm
- net GND: track 276.6 -> 345.9 mm, vias 9 -> 16
- net ESP_GPIO0: track 0.00 -> 64.8 mm, vias 0 -> 2
- net Net-(U2-Pad26): track 118.3 -> 63.2 mm
- net FEEDBACK: track 0.00 -> 38.2 mm, vias 0 -> 2
- net V_GND: track 0.00 -> 36.6 mm, vias 0 -> 2
- net ESP_RESET: track 0.00 -> 33.5 mm
- net V_READ_HV: track 27.0 -> 0.00 mm, vias 1 -> 0
- net Net-(POT1-Pad3): track 0.00 -> 27.0 mm, vias 0 -> 1
- net CLK: track 125.7 -> 151.0 mm
- net DISP_SCL: track 15.4 -> 38.1 mm, vias 0 -> 2
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Other:
- board text added: "V2.1, 2016"
- board text removed: "V2.0, 2016"

Commit message: Production Version 2.1 with Gerber Files
Version Bittie
Other:
- board text added: "17GN7NR9frDcqeuPHYKypcb2sEdwLDrEQ"
- board text added: "Queen Bittie"
- board text removed: "Festina lente!"
