File: OpenDropV3/DesignFiles/OpenDropV3.kicad_pcb (KiCad board)
At the start: 2 copper layers, 100 x 112 mm, 257 parts, among them J1 Conn_02x03_Odd_Even, J2 Conn_02x05_Odd_Even, J3 micro_USB, P1 CONN_01X01, P10 CONN_01X01, P11 CONN_01X01, P12 CONN_01X01, P13 ScrewPad1, P14 ScrewPad2, P15 ScrewPad3, P16 ScrewPad4, P2 ScrewPad4, P3 CONN_01X01, P7 CONN_01X01, P8 CONN_01X01, P9 CONN_01X01, SW1 SW_PUSH, SW2 SW_PUSH, SW3 SW_PUSH, SW5 SPST, T1 TK560P60Y, U1 MAX1771ESA, U10 AQY210EH, U11 AQY210EH, U12 AQY210EH, U13 AQY210EH, U14 TLV1117-33, U15 MCP41010, U16 74xx14, U2 HV507, U3 PAM8301, U4 HV507, U5 SAMD21G18B-A changed from SAM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, U6 MCP6002, U7 HCPL0534, U8 HCPL0534, U9 HCPL0534, Y1 32.765

Commit message: Improved design and corrected some errors. Allmost there
Parts:
- removed J3: micro_USB, GaudiLabsFootPrints:USB_Micro-B_FCI
- added C30: 100nF, Capacitors_SMD:C_0805, B.Cu at (110.4, 54.3)
- added C33: 100nF, Capacitors_SMD:C_0805, B.Cu at (117.0, 48.7)
- added C34: 100nF, Capacitors_SMD:C_0805, B.Cu at (124.7, 40.2)
- added G***: LOGO, GaudiLabsLogos:GitHubCat, B.Cu at (66.9, 132.2)
- added G***: LOGO, GaudiLabsLogos:AurynBio, B.Cu at (138.9, 90.8)
- added G***: LOGO, GaudiLabsLogos:ItsASynth, B.Cu at (75.4, 125.0)
- added G***: LOGO, GaudiLabsLogos:OSHW_OT3, B.Cu at (127.9, 131.9)
- added G***: LOGO, GaudiLabsLogos:GaudiLabs_8, B.Cu at (138.4, 98.9)
- added P4: CONN_PSEUDO_AC, Measurement_Points:Measurement_Point_Square-SMD-Pad_Small, B.Cu at (77.9, 86.4)
- added R12: 2.2k, Resistors_SMD:R_0805, B.Cu at (121.2, 53.8)
- added R13: 390, Resistors_SMD:R_0805, B.Cu at (121.2, 57.1)
- added REF***: KiCad-Logo2_6mm_SilkScreen, Symbols:KiCad-Logo2_6mm_SilkScreen, B.Cu at (138.9, 107.7)
- C21, C5: footprint Capacitors_SMD:C_0805 -> Capacitors_SMD:C_1206
- C32: value 22uF, 50V -> 100uF,35V; footprint GaudiLabsFootPrints:C_1913 -> Resistors_SMD:R_2512_HandSoldering
- FLUXL_10_1, FLUXL_10_8, FLUXL_11_1, FLUXL_11_8, FLUXL_12_1, FLUXL_12_8, FLUXL_13_1, FLUXL_13_8, FLUXL_14_1, FLUXL_14_8, FLUXL_3_1, FLUXL_3_8, FLUXL_4_1, FLUXL_4_8, FLUXL_5_1, FLUXL_5_8, FLUXL_6_1, FLUXL_6_8, FLUXL_7_1, FLUXL_7_8, FLUXL_8_1, FLUXL_8_8, FLUXL_9_1, FLUXL_9_8: footprint GaudiLabsFootPrints:FLUXL_PAD_2_75_top -> GaudiLabsFootPrints:FLUXPAD_2_75_4MIL_4_5_top
- FLUXL_10_2, FLUXL_10_3, FLUXL_10_4, FLUXL_10_5, FLUXL_10_6, FLUXL_10_7, FLUXL_11_2, FLUXL_11_3, FLUXL_11_4, FLUXL_11_5, FLUXL_11_6, FLUXL_11_7, FLUXL_12_2, FLUXL_12_3, FLUXL_12_4, FLUXL_12_5, FLUXL_12_6, FLUXL_12_7, FLUXL_13_2, FLUXL_13_3, FLUXL_13_4, FLUXL_13_5, FLUXL_13_6, FLUXL_13_7, FLUXL_14_2, FLUXL_14_3, FLUXL_14_4, FLUXL_14_5, FLUXL_14_6, FLUXL_14_7, FLUXL_15_2, FLUXL_15_7, FLUXL_2_2, FLUXL_2_7, FLUXL_3_2, FLUXL_3_3, FLUXL_3_4, FLUXL_3_5, FLUXL_3_6, FLUXL_3_7, FLUXL_4_2, FLUXL_4_3, FLUXL_4_4, FLUXL_4_5, FLUXL_4_6, FLUXL_4_7, FLUXL_5_2, FLUXL_5_3, FLUXL_5_4, FLUXL_5_5, FLUXL_5_6, FLUXL_5_7, FLUXL_6_2, FLUXL_6_3, FLUXL_6_4, FLUXL_6_5, FLUXL_6_6, FLUXL_6_7, FLUXL_7_2, FLUXL_7_3, FLUXL_7_4, FLUXL_7_5, FLUXL_7_6, FLUXL_7_7, FLUXL_8_2, FLUXL_8_3, FLUXL_8_4, FLUXL_8_5, FLUXL_8_6, FLUXL_8_7, FLUXL_9_2, FLUXL_9_3, FLUXL_9_4, FLUXL_9_5, FLUXL_9_6, FLUXL_9_7: footprint GaudiLabsFootPrints:FLUXL_PAD_2_75 -> GaudiLabsFootPrints:FLUXPAD_2_75_4MIL_4_5
- FLUXL_15_1, FLUXL_2_8: footprint GaudiLabsFootPrints:FLUXL_PAD_2_75_topright -> GaudiLabsFootPrints:FLUXPAD_2_75_4MIL_4_5_topright
- FLUXL_15_3, FLUXL_15_4, FLUXL_15_5, FLUXL_15_6, FLUXL_2_3, FLUXL_2_4, FLUXL_2_5, FLUXL_2_6: footprint GaudiLabsFootPrints:FLUXL_PAD_2_75_side -> GaudiLabsFootPrints:FLUXPAD_2_75_4MIL_4_5_side
- FLUXL_15_8, FLUXL_2_1: footprint GaudiLabsFootPrints:FLUXL_PAD_2_75_topleft -> GaudiLabsFootPrints:FLUXPAD_2_75_4MIL_4_5_topleft
- FLUXL_16_1, FLUXL_16_8, FLUXL_1_1, FLUXL_1_8: footprint GaudiLabsFootPrints:FLUXL_PAD_2_75_res3 -> GaudiLabsFootPrints:FLUXPAD_2_75_4MIL_4_5_res3
- FLUXL_16_2, FLUXL_16_7, FLUXL_1_2, FLUXL_1_7: footprint GaudiLabsFootPrints:FLUXL_PAD_2_75_res1 -> GaudiLabsFootPrints:FLUXPAD_2_75_4MIL_4_5_res1
- FLUXL_16_3, FLUXL_16_6, FLUXL_1_3, FLUXL_1_6: footprint GaudiLabsFootPrints:FLUXL_PAD_2_75_ref2 -> GaudiLabsFootPrints:FLUXPAD_2_75_4MIL_4_5_res2
- FLUXL_16_4, FLUXL_16_5, FLUXL_1_4, FLUXL_1_5: footprint GaudiLabsFootPrints:FLUXL_PAD_2_75_topleft -> GaudiLabsFootPrints:FLUXPAD_2_75_4MIL_4_5_res4
- FLUXL_16_4b1, FLUXL_16_5b1, FLUXL_1_4b1, FLUXL_1_5b1: footprint GaudiLabsFootPrints:FLUXL_PAD_2_75_topright -> GaudiLabsFootPrints:FLUXPAD_2_75_4MIL_4_5_res5
- J1: value Conn_02x03_Odd_Even -> USB_C_Receptacle; footprint Pin_Headers:Pin_Header_Straight_2x03_Pitch2.54mm_SMD -> Connectors_USB:USB_C_Receptacle_Amphenol_12401610E4-2A
- J2: footprint Pin_Headers:Pin_Header_Straight_2x05_Pitch1.27mm_SMD -> GaudiLabsFootPrints:Pin_Header_Straight_2x05_Pitch1.27mm_SMD
- SW3: footprint GaudiLabsFootPrints:PUSH_BUTTON_SMD -> GaudiLabsFootPrints:SW_SPST_KMS221GLFS
- U14: footprint TO_SOT_Packages_SMD:SOT-223 -> GaudiLabsFootPrints:SOT-223
- U5: footprint Housings_QFP:TQFP-48_7x7mm_Pitch0.5mm -> GaudiLabsFootPrints:TQFP-48_7x7mm_Pitch0.5mm
- moved J1 36.9 mm to (132.0, 35.9), turned to 0 degrees
- moved C26 11.7 mm to (109.5, 38.8), turned to 180 degrees
- moved C32 10.1 mm to (142.0, 38.8), turned to 270 degrees
- moved J2 8.08 mm to (95.9, 37.5)
- moved C21 4.37 mm to (124.7, 36.2)
- moved C20 4.32 mm to (105.8, 38.8)
- moved R6 3.07 mm to (122.6, 59.9), turned to 0 degrees
- moved C23 2.96 mm to (108.0, 36.8)
- moved C25 2.96 mm to (108.0, 34.8)
- moved Y1 2.47 mm to (111.3, 35.8), turned to 270 degrees
- moved U14 1.85 mm to (118.5, 37.3)
- moved C10 1.40 mm to (133.9, 43.4)
- moved C22 1.40 mm to (140.7, 61.7)
- moved C8 1.40 mm to (137.9, 43.4)
- moved R3 1.02 mm to (138.8, 40.2), turned to 90 degrees
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Connections:
- C11 pad 1: SPK -> Net-(C11-Pad1)
- U5 pad 10: Net-(U5-Pad10) -> JOY
- U5 pad 14: VSENS -> Net-(U5-Pad14)
- U5 pad 15: JOY -> Net-(U5-Pad15)
- U5 pad 16: V_SCK -> DISP_DC
- U5 pad 21: V_SI -> DISP_CS
- U5 pad 25: DISP_DC -> V_SI
- U5 pad 27: AC -> Net-(U5-Pad27)
- U5 pad 28: DISP_CS -> V_SCK
- U5 pad 47: Net-(U5-Pad47) -> SENS_PAD
- U5 pad 7: Net-(U5-Pad7) -> AC
- U5 pad 9: Net-(U5-Pad9) -> VSENS
Routing:
- net V_USB: track 160.6 -> 302.4 mm, vias 7 -> 6
- net SENS_PAD: track 0.00 -> 131.0 mm, vias 0 -> 2
- net GND: track 326.0 -> 361.3 mm, vias 40 -> 49
- net Net-(C11-Pad1): track 0.00 -> 13.8 mm, vias 0 -> 2
- net +3V3: track 296.9 -> 305.6 mm
- net JOY: track 164.1 -> 156.2 mm
- net AC: track 14.6 -> 21.7 mm, vias 0 -> 2
- net RX_LED: track 24.5 -> 31.2 mm
- net V_SCK: track 17.2 -> 12.0 mm
- net D+: track 38.2 -> 33.0 mm
- net SPK: track 18.6 -> 23.6 mm, vias 0 -> 2
- net Net-(C25-Pad2): track 12.2 -> 17.1 mm, vias 0 -> 2
- net DISP_DC: track 30.6 -> 25.9 mm
- net V_SI: track 16.7 -> 12.3 mm
- net Net-(FLUXL_1_4-Pad1): track 5.83 -> 9.38 mm
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- added copper zone on B.Cu, net +3V3
Other:
- net class Power: trace_width 0.2 -> 0.3; via_dia 0.6 -> 0.8; via_drill 0.4 -> 0.6
- board text added: "Q.C. PASSED"
- board text added: "RESET"
