File: OpenDropV3/DesignFiles/OpenDropV3.sch (KiCad schematic (older format))
At the start: 250 parts, among them J1 Conn_02x03_Odd_Even, J2 Conn_02x05_Odd_Even, J3 micro_USB, P1 CONN_01X01, P10 CONN_01X01, P11 CONN_01X01, P12 CONN_01X01, P13 ScrewPad1, P14 ScrewPad2, P15 ScrewPad3, P16 ScrewPad4, P2 ScrewPad4, P3 CONN_01X01, P7 CONN_01X01, P8 CONN_01X01, P9 CONN_01X01, SW1 SW_PUSH, SW2 SW_PUSH, SW3 SW_PUSH, SW5 SPST, T1 TK560P60Y, U1 MAX1771ESA, U10 AQY210EH, U11 AQY210EH, U12 AQY210EH, U13 AQY210EH, U14 TLV1117-33, U15 MCP41010, U16 74xx14, U2 HV507, U3 PAM8301, U4 HV507, U5 SAMD21G18B-A changed from SAM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, U6 MCP6002, U7 HCPL0534, U8 HCPL0534, U9 HCPL0534, Y1 32.765

Commit message: Improved design and corrected some errors. Allmost there
Parts:
- removed J1: Conn_02x03_Odd_Even, Pin_Headers:Pin_Header_Straight_2x03_Pitch2.54mm_SMD, symbol Conn_02x03_Odd_Even
- removed J3: micro_USB, GaudiLabsFootPrints:USB_Micro-B_FCI, symbol micro_USB
- added C30, C33, C34: 100nF, Capacitors_SMD:C_0805, symbol C
- added J1: USB_C_Receptacle, Connectors_USB:USB_C_Receptacle_Amphenol_12401610E4-2A, symbol USB_C_Receptacle
- added P4: CONN_PSEUDO_AC, Measurement_Points:Measurement_Point_Square-SMD-Pad_Small, symbol CONN_01X01
- added R12: 2.2k, Resistors_SMD:R_0805, symbol R
- added R13: 390, Resistors_SMD:R_0805, symbol R
- C21, C5: footprint Capacitors_SMD:C_0805 -> Capacitors_SMD:C_1206
- C32: value 22uF, 50V -> 100uF,35V; footprint GaudiLabsFootPrints:C_1913 -> Resistors_SMD:R_2512_HandSoldering
- FLUXL_10_1, FLUXL_10_8, FLUXL_11_1, FLUXL_11_8, FLUXL_12_1, FLUXL_12_8, FLUXL_13_1, FLUXL_13_8, FLUXL_14_1, FLUXL_14_8, FLUXL_3_1, FLUXL_3_8, FLUXL_4_1, FLUXL_4_8, FLUXL_5_1, FLUXL_5_8, FLUXL_6_1, FLUXL_6_8, FLUXL_7_1, FLUXL_7_8, FLUXL_8_1, FLUXL_8_8, FLUXL_9_1, FLUXL_9_8: footprint GaudiLabsFootPrints:FLUXL_PAD_2_75_top -> GaudiLabsFootPrints:FLUXPAD_2_75_4MIL_4_5_top
- FLUXL_10_2, FLUXL_10_3, FLUXL_10_4, FLUXL_10_5, FLUXL_10_6, FLUXL_10_7, FLUXL_11_2, FLUXL_11_3, FLUXL_11_4, FLUXL_11_5, FLUXL_11_6, FLUXL_11_7, FLUXL_12_2, FLUXL_12_3, FLUXL_12_4, FLUXL_12_5, FLUXL_12_6, FLUXL_12_7, FLUXL_13_2, FLUXL_13_3, FLUXL_13_4, FLUXL_13_5, FLUXL_13_6, FLUXL_13_7, FLUXL_14_2, FLUXL_14_3, FLUXL_14_4, FLUXL_14_5, FLUXL_14_6, FLUXL_14_7, FLUXL_15_2, FLUXL_15_7, FLUXL_2_2, FLUXL_2_7, FLUXL_3_2, FLUXL_3_3, FLUXL_3_4, FLUXL_3_5, FLUXL_3_6, FLUXL_3_7, FLUXL_4_2, FLUXL_4_3, FLUXL_4_4, FLUXL_4_5, FLUXL_4_6, FLUXL_4_7, FLUXL_5_2, FLUXL_5_3, FLUXL_5_4, FLUXL_5_5, FLUXL_5_6, FLUXL_5_7, FLUXL_6_2, FLUXL_6_3, FLUXL_6_4, FLUXL_6_5, FLUXL_6_6, FLUXL_6_7, FLUXL_7_2, FLUXL_7_3, FLUXL_7_4, FLUXL_7_5, FLUXL_7_6, FLUXL_7_7, FLUXL_8_2, FLUXL_8_3, FLUXL_8_4, FLUXL_8_5, FLUXL_8_6, FLUXL_8_7, FLUXL_9_2, FLUXL_9_3, FLUXL_9_4, FLUXL_9_5, FLUXL_9_6, FLUXL_9_7: footprint GaudiLabsFootPrints:FLUXL_PAD_2_75 -> GaudiLabsFootPrints:FLUXPAD_2_75_4MIL_4_5
- FLUXL_15_1, FLUXL_2_8: footprint GaudiLabsFootPrints:FLUXL_PAD_2_75_topright -> GaudiLabsFootPrints:FLUXPAD_2_75_4MIL_4_5_topright
- FLUXL_15_3, FLUXL_15_4, FLUXL_15_5, FLUXL_15_6, FLUXL_2_3, FLUXL_2_4, FLUXL_2_5, FLUXL_2_6: footprint GaudiLabsFootPrints:FLUXL_PAD_2_75_side -> GaudiLabsFootPrints:FLUXPAD_2_75_4MIL_4_5_side
- FLUXL_15_8, FLUXL_2_1: footprint GaudiLabsFootPrints:FLUXL_PAD_2_75_topleft -> GaudiLabsFootPrints:FLUXPAD_2_75_4MIL_4_5_topleft
- FLUXL_16_1, FLUXL_16_8, FLUXL_1_1, FLUXL_1_8: footprint GaudiLabsFootPrints:FLUXL_PAD_2_75_res3 -> GaudiLabsFootPrints:FLUXPAD_2_75_4MIL_4_5_res3
- FLUXL_16_2, FLUXL_16_7, FLUXL_1_2, FLUXL_1_7: footprint GaudiLabsFootPrints:FLUXL_PAD_2_75_res1 -> GaudiLabsFootPrints:FLUXPAD_2_75_4MIL_4_5_res1
- FLUXL_16_3, FLUXL_16_6, FLUXL_1_3, FLUXL_1_6: footprint GaudiLabsFootPrints:FLUXL_PAD_2_75_ref2 -> GaudiLabsFootPrints:FLUXPAD_2_75_4MIL_4_5_res2
- FLUXL_16_4, FLUXL_16_5, FLUXL_1_4, FLUXL_1_5: footprint GaudiLabsFootPrints:FLUXL_PAD_2_75_topleft -> GaudiLabsFootPrints:FLUXPAD_2_75_4MIL_4_5_res4
- FLUXL_16_4b1, FLUXL_16_5b1, FLUXL_1_4b1, FLUXL_1_5b1: footprint GaudiLabsFootPrints:FLUXL_PAD_2_75_topright -> GaudiLabsFootPrints:FLUXPAD_2_75_4MIL_4_5_res5
- J2: footprint Pin_Headers:Pin_Header_Straight_2x05_Pitch1.27mm_SMD -> GaudiLabsFootPrints:Pin_Header_Straight_2x05_Pitch1.27mm_SMD
- SW3: footprint GaudiLabsFootPrints:PUSH_BUTTON_SMD -> GaudiLabsFootPrints:SW_SPST_KMS221GLFS
- U14: footprint TO_SOT_Packages_SMD:SOT-223 -> GaudiLabsFootPrints:SOT-223
- U5: footprint Housings_QFP:TQFP-48_7x7mm_Pitch0.5mm -> GaudiLabsFootPrints:TQFP-48_7x7mm_Pitch0.5mm
Connections:
- net +3V3: now also C30.1, C33.2, C34.2
- net +5V: now also J1.A4 (VBUS), J1.A9 (VBUS), J1.B4 (VBUS), J1.B9 (VBUS)
- net AC: now also U5.7 (EXTINT8/AIN2/OAOUT1/SERCOM4PAD0/TC0WO0/CCL2IN2/PB08); no longer U5.27 (EXTINT2/X6/SERCOM1PAD2/SERCOM3PAD2/TC4WO0/TCC0WO2/ACCMP0/CCL0IN2/PA18)
- net D+: now also J1.A6 (D+), J1.B6 (D+)
- net D-: now also J1.A7 (D-), J1.B7 (D-)
- net DISP_CS: now also U5.21 (ACCMP0/TC2WO0/SERCOM4P0/SERCOM2P0/PA12); no longer U5.28 (EXTINT3/X7/SERCOM1PAD3/SERCOM3PAD3/TC4WO1/TCC0WO3/ACCMP1/CCL0OUT/PA19)
- net DISP_DC: now also U5.16 (EXTINT11/AIN19/X3Y9/SERCOM0PAD3/SERCOM2PAD3/TCC1WO1/TCC0WO3/GCLKIO5/CCL1OUT/PA11); no longer U5.25 (EXTINT0/X4/SERCOM1PAD0/SERCOM3PAD4/TCC2WO0/TCC0WO6/GCLKIO2/CCL0IN0/PA16)
- net GND: now also P13.1 (P1), C30.2, C33.1, C34.1, J1.A1 (GND), J1.A12 (GND), J1.B1 (GND), J1.B12 (GND), R13.2
- net JOY: now also U5.10 (EXTINT5EXTWAKE5/AIN5/AIN1/VOUT1/OAPOS2/SERCOM0PAD1/TCC0WO1/CCL0IN1/PA05); no longer U5.15 (EXTINT10/AIN18/X2Y8/SERCOM0PAD2/SERCOM2PAD2/TCC1WO0/TCC0WO2/GCLKIO4/CCL1IN2/PA10)
- net SPK: now also R12.2; no longer C11.1
- net VSENS: now also U5.9 (EXTINT4EXTWAKE4/VREFB/AIN4/AIN0/OAOUT2/SERCOM0PAD0/TCC0WO0/CCL0IN0/PA04); no longer U5.14 (EXTINT9/AIN17/X1Y7/SERCOM0PAD1/SERCOM2PAD1/TCC0WO1/TCC1WO3/CCL1IN1/PA09)
- net V_GND: now also P14.1 (P1); no longer P13.1 (P1)
- net V_SCK: now also U5.28 (EXTINT3/X7/SERCOM1PAD3/SERCOM3PAD3/TC4WO1/TCC0WO3/ACCMP1/CCL0OUT/PA19); no longer U5.16 (EXTINT11/AIN19/X3Y9/SERCOM0PAD3/SERCOM2PAD3/TCC1WO1/TCC0WO3/GCLKIO5/CCL1OUT/PA11)
- net V_SI: now also U5.25 (EXTINT0/X4/SERCOM1PAD0/SERCOM3PAD4/TCC2WO0/TCC0WO6/GCLKIO2/CCL0IN0/PA16); no longer U5.21 (ACCMP0/TC2WO0/SERCOM4P0/SERCOM2P0/PA12)
- net at FLUXL_1_4.1, FLUXL_1_4b1.1, U2.43 (HV_OUT_3): now also P4.1 (P1)
- net SENS_PAD: now reaches P16.1 (P1)
- net SENS_PAD: now also U5.47 (EXTINT2/AIN10/SERCOM5PAD0/TC2WO0/SUPCOUT1/CCL0OUT/PB02)
- new net: C11.1, R12.1, R13.1
Other:
- note added: "A1"
- note added: "A2 / LED? MKR\n"
- note added: "D1 / PWM2? MKR"
- note added: "LED? MKR\n"
- note added: "RXD0"
- note added: "TXD"
- note removed: "A1 / LED? MKR\n"
- note removed: "A4 / PWM2? MKR"
- moved on the sheet: C11, C14, C21, C22, C26, C27, C32, C5, J2, R15, R16, R17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
