File: OpenDropV3/OpenDropV3.kicad_pcb (KiCad board)
At the start: 2 copper layers, 100 x 112 mm, 270 parts, among them J1 USB_C_Receptacle, J2 Conn_02x05_Odd_Even, P1 CONN_01X01, P10 CONN_01X01, P11 CONN_01X01, P12 CONN_01X01, P13 ScrewPad1, P14 ScrewPad2, P15 ScrewPad3, P16 ScrewPad4, P2 ScrewPad4, P3 CONN_01X01, P4 CONN_PSEUDO_AC, P7 CONN_01X01, P8 CONN_01X01, P9 CONN_01X01, SW1 SW_PUSH, SW2 SW_PUSH, SW3 SW_PUSH, SW5 SPST, T1 TK560P60Y, U1 MAX1771ESA, U10 AQY210EH, U11 AQY210EH, U12 AQY210EH, U13 AQY210EH, U14 TLV1117-33, U15 MCP41010, U16 74xx14, U2 HV507, U3 PAM8301, U4 HV507, U5 SAMD21G18B-A changed from SAM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, U6 MCP6002, U7 HCPL0534, U8 HCPL0534, U9 HCPL0534, Y1 32.765

Commit message: Version 3.2 allmost done
Parts:
- removed the G*** at (127.9, 131.9)
- removed the G*** at (138.8, 98.9)
- added C37: 470pF, Capacitors_SMD:C_0805, B.Cu at (105.2, 73.5)
- added G***: LOGO, GaudiLabsLogos:OSHW_Logo_OpenDrop, B.Cu at (127.9, 131.9)
- added G***: LOGO, GaudiLabsLogos:GaudiLabs_12, B.Cu at (139.3, 99.5)
- added JS2: JoystickSMD_SKRH, GaudiLabsFootPrints:SKRHABE010, F.Cu at (100.0, 136.9)
- added R14: 0k, Resistors_SMD:R_0805, B.Cu at (109.5, 80.1)
- added R23: 0k, Resistors_SMD:R_0805, B.Cu at (111.6, 80.1)
- added R24: 0k, Resistors_SMD:R_0805, B.Cu at (113.8, 76.6)
- added R25: 0k, Resistors_SMD:R_0805, B.Cu at (111.6, 76.6)
- added R26: 0k, Resistors_SMD:R_0805, B.Cu at (107.3, 80.1)
- added R27: 0k, Resistors_SMD:R_0805, B.Cu at (64.1, 75.1)
- added R28: 0k, Resistors_SMD:R_0805, B.Cu at (65.4, 72.1)
- added R29: 680k?, Resistors_SMD:R_0805, B.Cu at (94.1, 57.5)
- added R46: 5k, Resistors_SMD:R_0805, B.Cu at (131.6, 43.4)
- added REF**: Pad_0_3, GaudiLabsFootPrints:Pad_0_3, F.Cu at (141.5, 134.1)
- added REF**: Pad_0_3, GaudiLabsFootPrints:Pad_0_3, F.Cu at (140.6, 134.9)
- added REF**: Pad_0_3, GaudiLabsFootPrints:Pad_0_3, F.Cu at (140.6, 133.4)
- added REF**: Pad_0_3, GaudiLabsFootPrints:Pad_0_3, F.Cu at (142.3, 133.4)
- C1, C32: footprint Resistors_SMD:R_2512_HandSoldering -> GaudiLabsFootPrints:C_2512_HandSoldering
- C21, C5: value 10uF -> 22uF
- R39: value 2.2k -> 5.6k
- moved U10 16.0 mm to (70.3, 66.1)
- moved R45 14.0 mm to (72.5, 73.4), turned to 0 degrees
- moved SW3 6.55 mm to (146.4, 49.3)
- moved R18 6.30 mm to (108.1, 133.8), turned to 0 degrees
- moved R48 5.33 mm to (77.9, 73.4)
- moved U11 5.33 mm to (75.6, 66.1)
- moved U12 5.33 mm to (86.3, 66.1)
- moved U13 5.33 mm to (80.9, 66.1)
- moved R51 4.57 mm to (82.4, 73.4)
- moved REF*** 4.33 mm to (139.2, 112.0)
- moved R49 4.06 mm to (86.5, 73.4), turned to 180 degrees
- moved R20 3.48 mm to (100.8, 138.0)
- moved R19 3.40 mm to (102.1, 133.8), turned to 0 degrees
- moved G*** 3.08 mm to (139.1, 87.7)
- moved C32 1.83 mm to (143.8, 39.1)
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Connections:
- C12 pad 1: VDD_C -> VDD_C2
- C12 pad 2: GND_C -> GND_C2
- C18 pad 2: GND_C -> GND_C2
- C35 pad 2: GND_C -> GND_C2
- J1 pad B5: Net-(J1-PadB5) -> Net-(J1-PadA5)
- P10 pad 1: BL_C -> BL_C2
- R35 pad 1: DI_C -> Net-(R24-Pad1)
- R39 pad 1: LE_C -> Net-(C37-Pad2)
- R42 pad 1: BL_C -> Net-(R25-Pad1)
- U16 pad 1: Net-(U16-Pad1) -> Net-(C28-Pad2)
- U16 pad 10: Net-(U12-Pad2) -> Net-(U13-Pad2)
- U16 pad 11: Net-(U16-Pad1) -> Net-(U16-Pad11)
- U16 pad 12: Net-(U10-Pad2) -> Net-(U12-Pad2)
- U16 pad 13: Net-(C28-Pad2) -> Net-(U16-Pad11)
- U16 pad 2: Net-(U11-Pad2) -> Net-(U10-Pad2)
- U16 pad 5: Net-(U16-Pad1) -> Net-(U16-Pad11)
- U16 pad 6: Net-(U13-Pad2) -> Net-(U11-Pad2)
- U16 pad 8: Net-(U16-Pad1) -> Net-(U16-Pad11)
- U2 pad 29: BL_C -> BL_C2
- U2 pad 30: POL_C -> POL_C2
- U3 pad 4: V_USB -> +3V3
- U3 pad 5: V_USB -> +3V3
- U4 pad 31: VDD_C -> VDD_C2
- U4 pad 32: GND_C -> GND_C2
- U4 pad 33: GND_C -> GND_C2
- U4 pad 34: GND_C -> GND_C2
- U7 pad 6: LE_C -> Net-(C37-Pad2)
- U8 pad 6: BL_C -> Net-(R25-Pad1)
- U9 pad 7: DI_C -> Net-(R24-Pad1)
Routing:
- net GND_C: track 305.6 -> 122.0 mm, vias 10 -> 0
- net GND_C2: track 0.00 -> 175.9 mm
- net VDD_C2: track 0.00 -> 147.4 mm
- net VDD_C: track 311.0 -> 176.9 mm, vias 5 -> 0
- net BL_C: track 157.9 -> 49.9 mm, vias 2 -> 0
- net BL_C2: track 0.00 -> 88.4 mm
- net POL_C: track 146.9 -> 62.0 mm, vias 2 -> 0
- net POL_C2: track 0.00 -> 75.3 mm
- net LE_C: track 155.6 -> 128.4 mm, vias 2 -> 0
- net Net-(U16-Pad1): track 20.4 -> 0.00 mm, vias 4 -> 0
- net Net-(U16-Pad11): track 0.00 -> 18.2 mm, vias 0 -> 4
- net Net-(U10-Pad2): track 12.7 -> 29.2 mm
- net CLK_C: track 157.7 -> 142.8 mm, vias 2 -> 0
- net DI_C: track 57.0 -> 42.3 mm, vias 2 -> 0
- net GND: track 363.8 -> 378.0 mm, vias 49 -> 52
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Other:
- net class Default: trace_width 0.15 -> 0.2
