File: OpenDropV3/OpenDropV3.sch (KiCad schematic (older format))
At the start: 257 parts, among them J1 USB_C_Receptacle, J2 Conn_02x05_Odd_Even, P1 CONN_01X01, P10 CONN_01X01, P11 CONN_01X01, P12 CONN_01X01, P13 ScrewPad1, P14 ScrewPad2, P15 ScrewPad3, P16 ScrewPad4, P2 ScrewPad4, P3 CONN_01X01, P4 CONN_PSEUDO_AC, P7 CONN_01X01, P8 CONN_01X01, P9 CONN_01X01, SW1 SW_PUSH, SW2 SW_PUSH, SW3 SW_PUSH, SW5 SPST, T1 TK560P60Y, U1 MAX1771ESA, U10 AQY210EH, U11 AQY210EH, U12 AQY210EH, U13 AQY210EH, U14 TLV1117-33, U15 MCP41010, U16 74xx14, U2 HV507, U3 PAM8301, U4 HV507, U5 SAMD21G18B-A changed from SAM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, U6 MCP6002, U7 HCPL0534, U8 HCPL0534, U9 HCPL0534, Y1 32.765

Commit message: Version 3.2 allmost done
Parts:
- added C37: 470pF, Capacitors_SMD:C_0805, symbol C
- added JS2: JoystickSMD_SKRH, GaudiLabsFootPrints:SKRHABE010, symbol JoystickSMD_SKRH
- added R14, R23, R24, R25, R26, R27, R28: 0k, Resistors_SMD:R_0805, symbol R
- added R29: 680k?, Resistors_SMD:R_0805, symbol R
- added R46: 5k, Resistors_SMD:R_0805, symbol R
- C1: footprint Resistors_SMD:R_2512_HandSoldering -> GaudiLabsFootPrints:C_2512_HandSoldering
- C32: value 100uF,50V -> 100uF,35V; footprint Resistors_SMD:R_2512_HandSoldering -> GaudiLabsFootPrints:C_2512_HandSoldering
- R39: value 2.2k -> 5.6k
Connections:
- net +3V3: now also U3.4 (~SD), U3.5 (VDD)
- net +5V: now also U16.14 (VCC); no longer U16.14 (VCC), U3.4 (~SD), U3.5 (VDD)
- net BL_C: now also R23.1, R25.2; no longer P10.1 (P1), R42.1, U2.29 (BL), U8.6 (COLLECTOR)
- net DI_C: now also R24.2; no longer R35.1, U9.7 (COLLECTOR)
- net GND: now also U16.7 (GND), JS2.5 (Common), R29.1, R46.2; no longer U16.7 (GND)
- net GND_C: now also R28.1; no longer C12.2, C18.2, C35.2, U4.32 (DIR), U4.33 (GND), U4.34 (HVGND)
- net JOY: now also JS2.4 (B_(right))
- net LE_C: now also R26.2; no longer R39.1, U7.6 (COLLECTOR)
- net POL_C: now also R14.1; no longer U2.30 (POL)
- net SW3: now also JS2.2 (Center)
- net VDD_C: now also C37.1, R27.2; no longer C12.1, U4.31 (VDD)
- net at JS1.1 (A_(up)), R21.1: now also JS2.1 (A_(up))
- net at JS1.2 (B_(left)), R20.1, R21.2: now also JS2.3 (C_(left))
- net at JS1.3 (C_(down)), R19.1, R20.2: now also JS2.6 (D_(down))
- net at U11.2: now also U16.6; no longer U16.2
- net at U10.2: now also U16.2; no longer U16.12
- net at U12.2: now also U16.12; no longer U16.10
- net at U13.2: now also U16.10; no longer U16.6
- net at C28.2, D2.2 (A), R10.2: now also U16.1; no longer U16.13
- net at C31.2, R11.1, U16.3: now also R29.2
- net at J1.A5 (CC1): now also J1.B5 (CC2), R46.1
- new net: R24.1, R35.1, U9.7 (COLLECTOR)
- new net: C37.2, R26.1, R39.1, U7.6 (COLLECTOR)
- new net: R25.1, R42.1, U8.6 (COLLECTOR)
- new net: U16.11, U16.13, U16.5, U16.8
- new net BL_C2: P10.1 (P1), R23.2, U2.29 (BL)
- new net GND_C2: C12.2, C18.2, C35.2, R28.2, U4.32 (DIR), U4.33 (GND), U4.34 (HVGND)
- new net POL_C2: R14.2, U2.30 (POL)
- new net VDD_C2: C12.1, R27.1, U4.31 (VDD)
Other:
- moved on the sheet: C12, C13, JS1, R18, R19, R20, R21, R32, R33, R36, R37, R38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
