File: OpenDropV3/Electronics/KiCad_Files/OpenDropV3.kicad_pcb (KiCad board)
At the start: 2 copper layers, 100 x 112 mm, 286 parts, among them J1 USB_C_Receptacle, J2 Conn_02x05_Odd_Even, P1 CONN_01X01, P10 CONN_01X01, P11 CONN_01X01, P12 CONN_01X01, P13 ScrewPad1, P14 ScrewPad2, P15 ScrewPad3, P16 ScrewPad4, P2 ScrewPad4, P3 CONN_01X01, P4 CONN_PSEUDO_AC, P7 CONN_01X01, P8 CONN_01X01, P9 CONN_01X01, SW1 SW_PUSH, SW2 SW_PUSH, SW3 SW_PUSH, SW5 SPST, T1 TK560P60Y, U1 MAX1771ESA, U10 AQY210EH, U11 AQY210EH, U12 AQY210EH, U13 AQY210EH, U14 TLV1117-33, U15 MCP41010, U16 74xx14, U2 HV507, U3 PAM8301, U4 HV507, U5 SAMD21G18B-A changed from SAM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, U6 MCP6002, U7 HCPL0534, U8 HCPL0534, U9 HCPL0534, Y1 32.765

Commit message: Production Files V3_2 This is it.
Parts:
- added REF**: Fiducial_1mm_Dia_2.54mm_Outer_CopperBottom, Fiducials:Fiducial_1mm_Dia_2.54mm_Outer_CopperBottom, F.Cu at (157.0, 36.0)
- added REF**: drillhole_0.3, GaudiLabsFootPrints:drillhole_0_5, F.Cu at (150.3, 39.0)
- added REF**: Fiducial_1mm_Dia_2.54mm_Outer_CopperBottom, Fiducials:Fiducial_1mm_Dia_2.54mm_Outer_CopperBottom, F.Cu at (157.0, 138.0)
- added REF**: drillhole_0.3, GaudiLabsFootPrints:drillhole_0_5, F.Cu at (150.3, 39.8)
- added REF**: drillhole_0.3, GaudiLabsFootPrints:drillhole_0_5, F.Cu at (49.7, 39.0)
- added REF**: drillhole_0.3, GaudiLabsFootPrints:drillhole_0_5, F.Cu at (150.3, 40.6)
- added REF**: drillhole_0.3, GaudiLabsFootPrints:drillhole_0_5, F.Cu at (150.3, 41.4)
- added REF**: drillhole_0.3, GaudiLabsFootPrints:drillhole_0_5, F.Cu at (150.3, 42.2)
- added REF**: drillhole_0.3, GaudiLabsFootPrints:drillhole_0_5, F.Cu at (150.3, 43.0)
- added REF**: drillhole_0.3, GaudiLabsFootPrints:drillhole_0_5, F.Cu at (150.3, 123.0)
- added REF**: drillhole_0.3, GaudiLabsFootPrints:drillhole_0_5, F.Cu at (150.3, 123.8)
- added REF**: drillhole_0.3, GaudiLabsFootPrints:drillhole_0_5, F.Cu at (150.3, 124.6)
- added REF**: drillhole_0.3, GaudiLabsFootPrints:drillhole_0_5, F.Cu at (150.3, 125.4)
- added REF**: Fiducial_1mm_Dia_2.54mm_Outer_CopperBottom, Fiducials:Fiducial_1mm_Dia_2.54mm_Outer_CopperBottom, F.Cu at (43.0, 137.0)
- added REF**: drillhole_0.3, GaudiLabsFootPrints:drillhole_0_5, F.Cu at (150.3, 126.2)
- added REF**: drillhole_0.3, GaudiLabsFootPrints:drillhole_0_5, F.Cu at (150.3, 127.0)
- added REF**: drillhole_0.3, GaudiLabsFootPrints:drillhole_0_5, F.Cu at (49.7, 39.8)
- added REF**: drillhole_0.3, GaudiLabsFootPrints:drillhole_0_5, F.Cu at (49.7, 40.6)
- added REF**: drillhole_0.3, GaudiLabsFootPrints:drillhole_0_5, F.Cu at (49.7, 41.4)
- added REF**: drillhole_0.3, GaudiLabsFootPrints:drillhole_0_5, F.Cu at (49.7, 42.2)
- added REF**: drillhole_0.3, GaudiLabsFootPrints:drillhole_0_5, F.Cu at (49.7, 43.0)
- added REF**: drillhole_0.3, GaudiLabsFootPrints:drillhole_0_5, F.Cu at (49.7, 123.0)
- added REF**: drillhole_0.3, GaudiLabsFootPrints:drillhole_0_5, F.Cu at (49.7, 123.8)
- added REF**: drillhole_0.3, GaudiLabsFootPrints:drillhole_0_5, F.Cu at (49.7, 124.6)
- added REF**: Fiducial_1mm_Dia_2.54mm_Outer_CopperBottom, Fiducials:Fiducial_1mm_Dia_2.54mm_Outer_CopperBottom, F.Cu at (43.0, 36.0)
- added REF**: drillhole_0.3, GaudiLabsFootPrints:drillhole_0_5, F.Cu at (49.7, 125.4)
- added REF**: drillhole_0.3, GaudiLabsFootPrints:drillhole_0_5, F.Cu at (49.7, 126.2)
- added REF**: drillhole_0.3, GaudiLabsFootPrints:drillhole_0_5, F.Cu at (49.7, 127.0)
- added REF**: Fiducial_1mm_Dia_2.54mm_Outer_CopperBottom, Fiducials:Fiducial_1mm_Dia_2.54mm_Outer_CopperBottom, B.Cu at (43.0, 137.0)
- added REF**: Fiducial_1mm_Dia_2.54mm_Outer_CopperBottom, Fiducials:Fiducial_1mm_Dia_2.54mm_Outer_CopperBottom, B.Cu at (43.0, 36.0)
- added REF**: Fiducial_1mm_Dia_2.54mm_Outer_CopperBottom, Fiducials:Fiducial_1mm_Dia_2.54mm_Outer_CopperBottom, B.Cu at (157.0, 138.0)
- added REF**: Fiducial_1mm_Dia_2.54mm_Outer_CopperBottom, Fiducials:Fiducial_1mm_Dia_2.54mm_Outer_CopperBottom, B.Cu at (157.0, 36.0)
Other:
- board size 100 x 112 mm -> 124 x 112 mm
