File: OpenDropV4/PCB/OpenDropV4/OpenDropV4.kicad_pcb (KiCad board)
At the start: 2 copper layers, 124 x 115.4 mm, 162 parts, among them J1 USB_C_Receptacle, J2 Conn_02x05_Odd_Even, J2 FFC_MOLEX_EASYON_05mm_24, J3 Conn_01x24_Female, P1 CONN_01X01, P12 CONN_01X01, P13 ScrewPad1, P14 ScrewPad2, P15 ScrewPad3, P16 ScrewPad4, P2 ScrewPad4, P3 CONN_01X01, P7 CONN_01X01, SW1 SW_PUSH, SW2 SW_PUSH, SW3 SW_PUSH, SW5 SPST, T1 TK560P60Y, U1 MAX1771ESA, U10 AQY210EH, U11 AQY210EH, U12 AQY210EH, U13 AQY210EH, U14 TLV1117-33, U15 MCP41010, U16 74xx14, U3 PAM8301, U5 SAMD21G18B-A changed from SAM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, U6 MCP6002, U7 HCPL0534, U8 HCPL0534, U9 HCPL0534, Y1 32.765

Commit message: Ready for second prototype round its not a synth
Parts:
- removed C32: 100uF,35V, GaudiLabsFootPrints:C_2512_HandSoldering
- removed the J2 at (100.0, 85.0)
- removed the REF** at (158.8, 169.4)
- removed the REF** at (158.8, 167.9)
- removed the REF** at (160.4, 167.9)
- removed the REF** at (159.6, 168.6)
- added REF**: MountingHole_2.7mm, MountingHole:MountingHole_2.7mm, F.Cu at (56.0, 123.4)
- added REF**: MountingHole_2.7mm, MountingHole:MountingHole_2.7mm, F.Cu at (102.4, 123.4)
- added REF**: MountingHole_2.7mm, MountingHole:MountingHole_2.7mm, F.Cu at (143.1, 123.4)
- C1: value 100uF, 35V -> 100uF, 6.3V; footprint GaudiLabsFootPrints:C_2512_HandSoldering -> Capacitor_SMD:C_1206_3216Metric
- C18, C4: footprint Capacitors_SMD:c_elec_10x10 -> Capacitor_SMD:C_Elec_8x10.2
- C19: value 22uF, 50V -> 100uF, 6.3V; footprint Capacitors_SMD:c_elec_6.3x5.8 -> Capacitor_SMD:C_1206_3216Metric
- C21, C5: value 22uF -> 100uF, 6.3V
- C35, C6: footprint GaudiLabsFootPrints:C_1913 -> Capacitor_SMD:C_1812_4532Metric_Pad1.30x3.40mm_HandSolder
- LED1, LED2, LED3: footprint LEDs:LED-0805 -> LED_SMD:LED_0603_1608Metric
- U7, U8, U9: value HCPL0534 -> ACPL-024L-000E
- moved G*** 6.63 mm to (131.2, 136.8)
- moved REF*** 5.58 mm to (67.2, 122.4)
- moved G*** 4.98 mm to (67.2, 116.0)
- moved G*** 4.07 mm to (134.3, 120.3)
- moved G*** 2.59 mm to (75.4, 129.0)
- moved C1 2.18 mm to (88.5, 38.5)
- moved C19 2.04 mm to (89.6, 56.1), turned to 270 degrees
- moved REF** 1.00 mm to (147.0, 130.0) (x2)
- moved REF** 1.00 mm to (53.0, 130.0) (x2)
- moved C18 0.67 mm to (59.0, 61.3), turned to 0 degrees
- moved C4 0.56 mm to (59.0, 39.1), turned to 180 degrees
- moved C6 0.38 mm to (67.7, 42.5)
- moved C5 0.12 mm to (139.8, 36.1)
Routing:
- net GND: track 317.9 -> 357.5 mm, vias 56 -> 58
- net V_USB: track 304.3 -> 286.3 mm
- net (no net): track 14.2 -> 0.00 mm
- net Net-(SP1-Pad1): track 151.5 -> 161.8 mm
- net Net-(SP1-Pad2): track 152.8 -> 162.7 mm
- net JOY: track 162.3 -> 171.9 mm
- net SW2: track 145.6 -> 155.0 mm
- net SW3: track 181.3 -> 190.2 mm
- net SW1: track 189.5 -> 198.3 mm
- net +3V3: track 336.6 -> 344.4 mm
- net VDD_C: track 165.7 -> 158.9 mm
- net GND_C: track 153.3 -> 147.7 mm
- net V_HV: track 43.7 -> 46.6 mm
- net SENS_PAD: track 73.9 -> 75.6 mm
- net Net-(D2-Pad1): track 18.0 -> 19.6 mm
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Other:
- board text added: "Driver Board"
- board text removed: "Community Coordinator: Eugenio Battaglia"
