File: OpenDropV4/PCB/OpenDropV4/OpenDropV4.sch (KiCad schematic (older format))
At the start: 112 parts, among them J1 USB_C_Receptacle, J2 Conn_02x05_Odd_Even, J3 Conn_01x24_Female, P1 CONN_01X01, P12 CONN_01X01, P13 ScrewPad1, P14 ScrewPad2, P15 ScrewPad3, P16 ScrewPad4, P2 ScrewPad4, P3 CONN_01X01, P7 CONN_01X01, SW1 SW_PUSH, SW2 SW_PUSH, SW3 SW_PUSH, SW5 SPST, T1 TK560P60Y, U1 MAX1771ESA, U10 AQY210EH, U11 AQY210EH, U12 AQY210EH, U13 AQY210EH, U14 TLV1117-33, U15 MCP41010, U16 74xx14, U3 PAM8301, U5 SAMD21G18B-A changed from SAM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, U6 MCP6002, U7 HCPL0534, U8 HCPL0534, U9 HCPL0534, Y1 32.765

Commit message: Ready for second prototype round its not a synth
Parts:
- removed C32: 100uF,35V, GaudiLabsFootPrints:C_2512_HandSoldering, symbol OpenDropV4-rescue:CP
- C1: value 100uF, 35V -> 100uF, 6.3V; footprint GaudiLabsFootPrints:C_2512_HandSoldering -> Capacitor_SMD:C_1206_3216Metric
- C18, C4: footprint Capacitors_SMD:c_elec_10x10 -> Capacitor_SMD:C_Elec_8x10.2
- C19: value 22uF, 50V -> 100uF, 6.3V; footprint Capacitors_SMD:c_elec_6.3x5.8 -> Capacitor_SMD:C_1206_3216Metric
- C21, C5: value 22uF -> 100uF, 6.3V
- C35, C6: footprint GaudiLabsFootPrints:C_1913 -> Capacitor_SMD:C_1812_4532Metric_Pad1.30x3.40mm_HandSolder
- LED1, LED2, LED3: footprint LEDs:LED-0805 -> LED_SMD:LED_0603_1608Metric
- U7, U8, U9: value HCPL0534 -> ACPL-024L-000E
Other:
- moved on the sheet: C10, C14, C20, C21, C22, C23, C24, C25, C26, C27, C30, C33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
