File: OpenDropV4/Electronics/OpenDropV4/OpenDropV4.sch (KiCad schematic (older format))
At the start: 111 parts, among them J1 USB_C_Receptacle, J2 Conn_02x05_Odd_Even, J3 Conn_01x24_Female, P1 CONN_01X01, P12 CONN_01X01, P13 ScrewPad1, P14 ScrewPad2, P15 ScrewPad3, P16 ScrewPad4, P2 ScrewPad4, P3 CONN_01X01, P7 CONN_01X01, SW1 SW_PUSH, SW2 SW_PUSH, SW3 SW_PUSH, SW5 SPST, T1 TK560P60Y, U1 MAX1771ESA, U10 AQY210EH, U11 AQY210EH, U12 AQY210EH, U13 AQY210EH, U14 TLV1117-33, U15 MCP41010, U16 74xx14, U3 PAM8301, U5 SAMD21G18B-A changed from SAM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, U6 MCP6002, U7 ACPL-024L-000E, U8 ACPL-024L-000E, U9 ACPL-024L-000E, Y1 32.765

Commit message: Updated to V4.1 in Software and Electronics
Parts:
- added D4: PESD5V0L5UY, Package_TO_SOT_SMD:SOT-363_SC-70-6, symbol Power_Protection:PESD5V0L5UY
- added D5: D_TVS, GaudiLabsFootPrints:DO-214AA, symbol Device:D_TVS
- added FB1, FB2, FB3, FB4, FB5, FB6, FB8: Ferrite_Bead_Small, Inductor_SMD:L_0603_1608Metric, symbol Device:Ferrite_Bead_Small
- added R14: 10k, Resistor_SMD:R_0805_2012Metric, symbol OpenDropV4-rescue:R
- added R7: 6.8k, Resistor_SMD:R_0805_2012Metric, symbol OpenDropV4-rescue:R
- U15: value MCP41010 -> MCP41050
Connections:
- net BL_C: now also D4.6 (K5), FB4.1; no longer U8.6 (COLLECTOR)
- net CLK_C: now also D4.3 (K2), FB1.1; no longer U7.7 (COLLECTOR)
- net DIG1: now also U5.13 (NMI/AIN16/X0Y6/SERCOM0PAD0/SERCOM2PAD0/TCC0WO0/TCC1WO2/CCL1IN0/PA08); no longer U5.15 (EXTINT10/AIN18/X2Y8/SERCOM0PAD2/SERCOM2PAD2/TCC1WO0/TCC0WO2/GCLKIO4/CCL1IN2/PA10)
- net DI_C: now also D4.4 (K3), FB5.1; no longer U9.7 (COLLECTOR)
- net GND: now also R14.2
- net GND_C: now also D4.2 (A), D5.2 (A2)
- net LE: now also U5.15 (EXTINT10/AIN18/X2Y8/SERCOM0PAD2/SERCOM2PAD2/TCC1WO0/TCC0WO2/GCLKIO4/CCL1IN2/PA10); no longer U5.13 (NMI/AIN16/X0Y6/SERCOM0PAD0/SERCOM2PAD0/TCC0WO0/TCC1WO2/CCL1IN0/PA08)
- net LE_C: now also D4.1 (K1), FB3.1; no longer C37.2, U7.6 (COLLECTOR)
- net POL_C: now also D4.5 (K4), FB2.1; no longer U8.7 (COLLECTOR)
- net VDD_C: now also D5.1 (A1), FB6.2; no longer J3.18 (Pin_18)
- net V_HV_C: now also FB8.2; no longer J3.20 (Pin_20)
- net at C1.1, C2.1, L1.1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: now also R7.1
- net V_USB_SENS: now reaches U5.47 (EXTINT2/AIN10/SERCOM5PAD0/TC2WO0/SUPCOUT1/CCL0OUT/PB02)
- net V_USB_SENS: now also R14.1, R7.2
- new net: FB1.2, U7.7 (COLLECTOR)
- new net: C37.2, FB3.2, U7.6 (COLLECTOR)
- new net: FB2.2, U8.7 (COLLECTOR)
- new net: FB5.2, U9.7 (COLLECTOR)
- new net: FB4.2, U8.6 (COLLECTOR)
- new net: FB6.1, J3.18 (Pin_18)
- new net: FB8.1, J3.20 (Pin_20)
Other:
- note added: "1.5V"
- note added: "50k"
- note added: "VOUT = 1.5 x (R2/R1 +1)"
- note removed: "10k"
- note removed: "65-260VDC"
- moved on the sheet: J3, R34, R40, R41, U8B, U9A, U9B
